File: STM32-PCb/STM32-PCb.kicad_sch (KiCad schematic)
At the start: 24 parts, among them J1 Conn_Coaxial, J2 Conn_ARM_SWD_TagConnect_TC2030, U1 STM32WB55CEUx, X1 32MHz, X2 32kHz768

Commit message: finished schematic added USB, LDO, BNO55, and stm mems sensors
Parts:
- added C16, C19, C20, C23, C24, C25, C26, C27: 100n, symbol Device:C
- added C17, C18: 4u7, symbol Device:C
- added C21, C22: 22p, symbol Device:C
- added D1: LED, symbol Device:LED
- added J3: Conn_01x04_Socket, Connector_Molex:Molex_MicroClasp_55932-0410_1x04_P2.00mm_Vertical, symbol Connector:Conn_01x04_Socket
- added J4: USB_C_Receptacle_USB2.0_NO_SBU, symbol josh-connector:USB_C_Receptacle_USB2.0_NO_SBU
- added R1, R3, R4: 5k1, symbol Device:R
- added R10, R11, R12, R13, R14, R15, R5, R6, R7, R8, R9: 10K, symbol Device:R
- added R16, R17, R18: 220R, symbol Device:R
- added R2: 100R, symbol Device:R
- added SW1: SW_Push, symbol Switch:SW_Push
- added U2: USBLC6-2SC6, Package_TO_SOT_SMD:SOT-23-6, symbol Power_Protection:USBLC6-2SC6
- added U3: MIC5365-3.3YD5, Package_TO_SOT_SMD:SOT-23-5, symbol Regulator_Linear:MIC5365-3.3YD5
- added U4: BNO055, Package_LGA:LGA-28_5.2x3.8mm_P0.5mm, symbol Sensor_Motion:BNO055
- added U5: LIS331HH, Package_LGA:LGA-12_2x2mm_P0.5mm, symbol Sensor_Motion:LIS331HH
- added U6: LSM6DS3, Package_LGA:LGA-14_3x2.5mm_P0.5mm_LayoutBorder3x4y, symbol Sensor_Motion:LSM6DS3
- added X3: 32kHz768, symbol Device:Crystal
Connections:
- net +3V3: now also C18.1, C20.1, C23.1, C24.1, C25.1, C26.1, C27.1, J3.4 (Pin_4), R12.2, R13.1, R14.2, R15.1, R8.2, R9.1, SW1.2, U3.5 (VOUT), U4.28 (VDDIO), U4.3 (VDD), U4.4 (~{BOOT_LOAD_PIN}), U5.1 (Vdd_IO), U5.14 (Vdd), U5.15 (Vdd), U5.8 (~{CS}), U6.12 (CS), U6.5 (VDDIO), U6.8 (VDD)
- net GND: now also C16.2, C17.2, C18.2, C19.2, C20.2, C21.2, C22.2, C23.2, C24.2, C25.2, C26.2, C27.2, J3.1 (Pin_1), J4.A1 (GND), J4.S1 (SHIELD), J4.S2 (SHIELD), J4.S3 (SHIELD), J4.S4 (SHIELD), R1.2, R10.2, R11.2, R18.2, R3.2, R4.2, R5.2, R6.1, R7.2, U2.2 (GND), U3.2 (GND), U4.18 (COM2), U4.2 (GND), U4.25 (GNDIO), U5.10 (GND), U5.12 (GND), U5.13 (GND), U5.16 (GND), U5.5 (GND), U6.6 (GND), U6.7 (GND)
- net UART_TX: now reaches U1.11 (PA2)
- net UART_TX: now also R16.2
- net UART_RX: now reaches U1.12 (PA3)
- net UART_RX: now also R17.1
- net I2C1_SCL: now reaches U1.15 (PA6)
- net I2C1_SCL: now also R12.1, R14.1, R9.2, U4.19 (COM1), U5.4 (SCL/SPC), U6.13 (SCL)
- net I2C1_SDA: now reaches U1.16 (PA7)
- net I2C1_SDA: now also R13.2, R15.2, R8.1, U4.20 (COM0), U5.6 (SDA/SDI), U6.14 (SDA)
- net at U1.18 (PA9): now also D1.2 (A)
- net USB_D-: now reaches U1.37 (PA11)
- net USB_D-: now also J4.A7 (D-), J4.B7 (D-), U2.1 (I/O1), U2.6 (I/O1)
- net USB_D+: now reaches U1.38 (PA12)
- net USB_D+: now also J4.A6 (D+), J4.B6 (D+), U2.3 (I/O2), U2.4 (I/O2)
- net BOOT_M: now reaches U1.4 (PH3)
- net BOOT_M: now also C16.1, R1.1, R2.1
- new net: D1.1 (K), R18.1
- new net: C21.1, U4.27 (XIN32), X3.1
- new net: R10.1, U5.7 (SA0/SDO)
- new net: R7.1, U4.17 (COM3)
- new net: C22.1, U4.26 (XOUT32), X3.2
- new net: R6.2, U4.5 (PS1)
- new net: R5.1, U4.6 (PS0)
- new net: C19.1, U4.9 (CAP)
- new net: R2.2, SW1.1
- new net: R11.1, U6.1 (SDO/SA0)
- new net UART_RXC: J3.2 (Pin_2), R17.2
- new net UART_TXC: J3.3 (Pin_3), R16.1
- new net USB_CC1: J4.A5 (CC1), R4.1
- new net USB_CC2: J4.B5 (CC2), R3.1
- new net VBUS: C17.1, J4.A4 (VBUS), U2.5 (VBUS), U3.1 (VIN), U3.3 (EN)
- no-connect marks 0 -> 9
Other:
- note added: "BLUETOOTH/RF"
- note added: "BNO55 all in one 9DOF IMU (I2C)"
- note added: "BOOT MODE & USR button"
- note added: "DEBUG"
- note added: "STM LIS331HH & LSM6DS3 combo for 9DOF sensing (I2C)"
- note added: "STM32WB55"
- note added: "USB 2.0 and VBUS"
- note added: "VBUS to 3.3 LDO"
- title: (none) -> STM32 BL and 9DOF test board
- moved on the sheet: C14, C15, J1, J2, L3, LPF1
